File: MLAB_MCU_pcb.kicad_sch (KiCad schematic)
At the start: 93 parts, among them J1 TBC05-02-1-G-G, J10 Conn_01x02_Pin, J11 Conn_02x06_Odd_Even, J12 Conn_02x06_Odd_Even, J13 Conn_01x02_Pin, J2 Input Header, J21 Conn_01x02_Pin, J22 Conn_01x02_Pin, J23 Conn_Coaxial, J24 Conn_Coaxial, J25 Conn_01x02_Pin, J26 Conn_01x02_Pin, J27 Conn_01x02_Pin, J28 232-5205-01, J3 Conn_Coaxial, J31 Conn_02x05_Odd_Even, J32 Conn_02x05_Odd_Even, J4 Conn_01x02_Pin, J5 Conn_01x02_Pin, J6 Conn_01x02_Pin, J7 Conn_01x03_Pin, J8 Conn_01x02_Pin, J9 Conn_Coaxial, U1 DSC1101DL5-020.0000, U2 TPS7A2012PDBVRG4, U3 TPS7A2033PDBVR, U4 24LC512, U5 INA4180A1

Commit message: Routing WIP
Parts:
- added H1, H2, H3, H4: MountingHole, MountingHole:MountingHole_3.2mm_M3, symbol Mechanical:MountingHole

Commit message: Routed
Connections:
- net GPIO2_ISO: now also J12.11 (Pin_11); no longer J12.12 (Pin_12)
- net GPIO3_ISO: now also J12.9 (Pin_9); no longer J12.10 (Pin_10)
- net GPIO4_ISO: now also J12.7 (Pin_7); no longer J12.8 (Pin_8)
- net GPIO5_ISO: now also J12.5 (Pin_5); no longer J12.6 (Pin_6)
- net GPIO6_ISO: now also J12.12 (Pin_12); no longer J12.11 (Pin_11)
- net GPIO7_ISO: now also J12.10 (Pin_10); no longer J12.9 (Pin_9)
- net GPIO8_ISO: now also J12.8 (Pin_8); no longer J12.7 (Pin_7)
- net GPIO9_ISO: now also J12.6 (Pin_6); no longer J12.5 (Pin_5)
Other:
- note added: "Short instead of R2 for the start"
- note removed: "Short instead of R7 for the start"
Changed lines of the file:
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@@
 		)
 	)
-	(text "Short instead of R7 for the start"
+	(text "Short instead of R2 for the start"
 		(exclude_from_sim no)
 		(at 81.788 235.458 0)
@@
 		)
 	)
-	(label "GPIO5_ISO"
+	(label "GPIO9_ISO"
 		(at 372.11 191.77 0)
 		(effects
@@
 		)
 	)
-	(label "GPIO8_ISO"
+	(label "GPIO4_ISO"
 		(at 342.9 194.31 0)
 		(effects
@@
 		)
 	)
-	(label "GPIO7_ISO"
+	(label "GPIO3_ISO"
 		(at 342.9 196.85 0)
 		(effects
@@
 		)
 	)
-	(label "GPIO9_ISO"
+	(label "GPIO5_ISO"
 		(at 342.9 191.77 0)
 		(effects
@@
 		)
 	)
-	(label "GPIO3_ISO"
+	(label "GPIO7_ISO"
 		(at 372.11 196.85 0)
 		(effects
@@
 		)
 	)
-	(label "GPIO2_ISO"
+	(label "GPIO6_ISO"
 		(at 372.11 199.39 0)
 		(effects
@@
 		)
 	)
-	(label "GPIO6_ISO"
+	(label "GPIO2_ISO"
 		(at 342.9 199.39 0)
 		(effects
@@
 		)
 	)
-	(label "GPIO4_ISO"
+	(label "GPIO8_ISO"
 		(at 372.11 194.31 0)
 		(effects

Commit message: Final changes and output files
Parts:
- J23, J24, J3, J9: footprint Connector_Coaxial:SMA_Amphenol_132134_Vertical -> 1_mlab_mcu_fp:SMA-J-P-X-ST-TH1-MKT
Changed lines of the file:
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@@
 			)
 		)
-		(property "Footprint" "Connector_Coaxial:SMA_Amphenol_132134_Vertical"
+		(property "Footprint" "1_mlab_mcu_fp:SMA-J-P-X-ST-TH1-MKT"
 			(at 87.63 198.12 0)
 			(hide yes)
@@
 			)
 		)
-		(property "Footprint" "Connector_Coaxial:SMA_Amphenol_132134_Vertical"
+		(property "Footprint" "1_mlab_mcu_fp:SMA-J-P-X-ST-TH1-MKT"
 			(at 191.77 40.64 0)
 			(hide yes)
@@
 			)
 		)
-		(property "Footprint" "Connector_Coaxial:SMA_Amphenol_132134_Vertical"
+		(property "Footprint" "1_mlab_mcu_fp:SMA-J-P-X-ST-TH1-MKT"
 			(at 287.02 151.13 0)
 			(hide yes)
@@
 			)
 		)
-		(property "Footprint" "Connector_Coaxial:SMA_Amphenol_132134_Vertical"
+		(property "Footprint" "1_mlab_mcu_fp:SMA-J-P-X-ST-TH1-MKT"
 			(at 285.75 40.64 0)
 			(hide yes)
